File: Mark_III/RGB_Amp/Kicad/Sega_MarkIII_RGB_Amp.kicad_sch (KiCad schematic)
At the start: 12 parts, among them IC1 THS7314D, J1 RGBS_Input, J2 RGBS_Output

Commit message: New PCB layout
Parts:
- removed HOLE1: HOLE, MountingHole:MountingHole_3.2mm_M3_DIN965_Pad_TopOnly, symbol my_components:HOLE
- removed J1: RGBS_Input, Connector_PinHeader_2.54mm:PinHeader_1x06_P2.54mm_Horizontal, symbol Connector:Conn_01x06_Pin
- removed J2: RGBS_Output, Connector_PinHeader_2.54mm:PinHeader_1x05_P2.54mm_Horizontal, symbol Connector:Conn_01x05_Pin
- added H1: MountingHole_Pad, MountingHole:MountingHole_3.2mm_M3_DIN965_Pad_TopBottom, symbol Mechanical:MountingHole_Pad
- added J1: RGBS Input, Connector_PinHeader_2.54mm:PinHeader_1x06_P2.54mm_Horizontal, symbol Connector_Generic:Conn_01x06
- added J2: RGBS Output, Connector_PinHeader_2.54mm:PinHeader_1x05_P2.54mm_Horizontal, symbol Connector_Generic:Conn_01x05
- added J3: RGBS Output, symbol Connector:DIN-8
Connections:
- net +5V: now also J1.5 (Pin_5)
- net GND: now also H1.1, J1.6 (Pin_6), J2.5 (Pin_5), J3.2
- net RED_{OUT}: now reaches R1.1, R7.1
- net RED_{OUT}: now also J2.2 (Pin_2), J3.7
- net BLUE_{OUT}: now reaches R3.1, R5.1
- net BLUE_{OUT}: now also J2.4 (Pin_4), J3.8
- net GREEN_{OUT}: now reaches R2.1, R6.1
- net GREEN_{OUT}: now also J2.3 (Pin_3), J3.4
- net SYNC_{OUT}: now reaches R4.1
- net SYNC_{OUT}: now also J2.1 (Pin_1), J3.6
- net BLUE renamed BLUE_{IN}
- net BLUE_{IN}: now also J1.4 (Pin_4)
- net GREEN renamed GREEN_{IN}
- net GREEN_{IN}: now also J1.3 (Pin_3)
- net RED renamed RED_{IN}
- net RED_{IN}: now also J1.2 (Pin_2)
- net SYNC renamed SYNC_{IN}
- net SYNC_{IN}: now also J1.1 (Pin_1)
- no-connect marks 0 -> 3
Other:
- title: Sega Mark II RGB Amplifier -> Sega Mark III RGB Amplifier
- moved on the sheet: C1, IC1, R1, R2, R3, R4, R5, R6, R7
