File: Mark_III/RGB_Amp/Kicad/Sega_MarkIII_RGB_Amp.kicad_pcb (KiCad board)
At the start: 2 copper layers, 26 x 29 mm, 12 parts, among them IC1 THS7314D, J1 RGBS_Input, J2 RGBS_Output

Commit message: New PCB layout
Parts:
- removed HOLE1: HOLE, MountingHole:MountingHole_3.2mm_M3_DIN965_Pad_TopOnly
- added H1: MountingHole_Pad, MountingHole:MountingHole_3.2mm_M3_DIN965_Pad_TopBottom, F.Cu at (120.7, 76.8)
- J1: value RGBS_Input -> RGBS Input
- J2: value RGBS_Output -> RGBS Output
- moved R7 128.1 mm to (125.1, 67.3)
- moved R6 128.0 mm to (125.1, 69.8)
- moved R5 127.9 mm to (125.1, 72.4)
- moved R1 127.3 mm to (121.0, 67.3)
- moved R2 127.2 mm to (121.0, 69.8)
- moved IC1 127.1 mm to (115.1, 69.8)
- moved R3 127.0 mm to (121.0, 72.4)
- moved J2 125.9 mm to (129.0, 66.0), turned to 0 degrees
- moved C1 122.6 mm to (113.4, 74.3), turned to 180 degrees
- moved J1 118.1 mm to (109.2, 77.5), turned to 180 degrees
- moved R4 118.1 mm to (123.2, 63.5), turned to 180 degrees
Connections:
- net /BLUE renamed /BLUE_{IN}
- net /GREEN renamed /GREEN_{IN}
- net /RED renamed /RED_{IN}
- net /SYNC renamed /SYNC_{IN}
- net Net-(J2-Pin_3) renamed GREEN_{OUT}
- C1 pad 1: /GND -> GND
- IC1 pad 5: /GND -> GND
- J1 pad 6: /GND -> GND
- J2 pad 1: /GND -> SYNC_{OUT}
- J2 pad 2: Net-(J2-Pin_2) -> RED_{OUT}
- J2 pad 4: Net-(J2-Pin_4) -> BLUE_{OUT}
- J2 pad 5: Net-(J2-Pin_5) -> GND
- R1 pad 1: Net-(J2-Pin_4) -> RED_{OUT}
- R3 pad 1: Net-(J2-Pin_2) -> BLUE_{OUT}
- R4 pad 1: Net-(J2-Pin_5) -> SYNC_{OUT}
- R5 pad 1: Net-(J2-Pin_2) -> BLUE_{OUT}
- R5 pad 2: /GND -> GND
- R6 pad 2: /GND -> GND
- R7 pad 1: Net-(J2-Pin_4) -> RED_{OUT}
- R7 pad 2: /GND -> GND
Routing:
- net Net-(J2-Pin_4): track 22.9 -> 0.00 mm
- net /BLUE_{IN}: track 19.2 -> 3.96 mm
- net Net-(J2-Pin_2): track 13.2 -> 0.00 mm
- net /+5V: track 17.5 -> 7.03 mm
- net GREEN_{OUT}: track 17.3 -> 7.48 mm
- net Net-(J2-Pin_5): track 9.65 -> 0.00 mm
- net /SYNC_{IN}: track 5.86 -> 13.5 mm
- net RED_{OUT}: track 0.00 -> 7.48 mm
- net BLUE_{OUT}: track 0.00 -> 7.48 mm
- net /GREEN_{IN}: track 9.58 -> 3.44 mm
- net SYNC_{OUT}: track 0.00 -> 5.83 mm
- net /RED_{IN}: track 8.38 -> 3.44 mm
- net Net-(IC1-CH.1_OUT): track 4.24 -> 2.46 mm
- net Net-(IC1-CH.2_OUT): track 3.82 -> 2.46 mm
- net GND: vias 0 -> 5
- added copper zone on B.Cu, net GND
- added copper zone on F.Cu, net GND
- removed copper zone on F.Cu, net /GND
Other:
- board size 26 x 29 mm -> 28.6 x 19.7 mm
- board text added: "1 2 3 4 5"
- board text added: "1 2 3 4 5 6"
- board text added: "1 = GND (DIN p2) 2 = BLUE (DIN p8) 3 = GREEN (DIN p4) 4 = RED (DIN p7) 5 = SYNC (DIN p6)"
- board text added: "1 = SYNC (VDP p29) 2 = RED (VDP p26) 3 = GREEN (VDP p27) 4 = BLUE (VDP p28) 5 = +5V 6 = GND"
- board text added: "Brett Hallen, Sept 2023/Nov 2025"
- board text added: "RGBS Input"
- board text added: "RGBS Output"
- board text added: "Sega Mark III RGB Amp. Board (Rev B)"
- board text removed: "P1 = GND (DIN p2) P2 = BLUE (DIN p8) P3 = GREEN (DIN p4) P4 = RED (DIN p7) P5 = SYNC (DIN p6)"
- board text removed: "P1 = SYNC (VDP p29) P2 = RED (VDP p26) P3 = GREEN (VDP p27) P4 = BLUE (VDP p28) P5 = +5V P6 = GND"

Commit message: Minor 5V track re-route
Routing:
- net /+5V: track 7.03 -> 5.98 mm
- net GND: vias 5 -> 6
Changed lines of the file:
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@@
+	)
+	(segment
+		(start 111.76 74.93)
+		(end 112.395 74.295)
+		(width 0.25)
+		(layer "F.Cu")
+		(net 4)
 	)
 	(segment
@@
 	(segment
 		(start 109.22 74.93)
-		(end 112.395 71.755)
+		(end 111.76 74.93)
 		(width 0.25)
 		(layer "F.Cu")
@@
 		(net 5)
 	)
+	(via
+		(at 110.925 73.495)
+		(size 0.8)
+		(drill 0.4)
+		(layers "F.Cu" "B.Cu")
+		(free yes)
+		(net 5)
+	)
