File: Mark_III/RGB_Amp_Internal/Kicad/Sega_MarkIII_RGB_Amp_Internal.kicad_sch (KiCad schematic)
At the start: 13 parts, among them IC1 THS7314D, J1 RGBS Input, J2 RGBS Output, J3 RGBS Output

Commit message: Refreshing design & repository
Other:
- title: Sega Mark III RGB Amplifier -> Sega Mark III RGB Amplifier (Internal)
Changed lines of the file:
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@@
 	(paper "A5")
 	(title_block
-		(title "Sega Mark III RGB Amplifier")
+		(title "Sega Mark III RGB Amplifier (Internal)")
 		(date "22/NOV/2025")
 		(rev "B")
